Commit message: Update body.stl; Add Gazebo plugins in URDF

File: knight_description/urdf/knight.urdf (robot description, URDF)
Before this commit: robot knight, 4 links, 3 joints
Links:
- added link imu_link; visual box size=0.015 0.015 0.015
- added link lidar_link; visual box size=0.015 0.015 0.015
- link base_link: mass 1 -> 4
- link left_wheel_link: mass 0.4 -> 0.5
- link right_wheel_link: mass 0.4 -> 0.5
Joints:
- added joint imu_joint: type fixed, parent base_link, child imu_link, origin xyz=0 0.140 0.026 rpy=0 0 0
- added joint lidar_joint: type fixed, parent base_link, child lidar_link, origin xyz=0 0 0.19 rpy=0 0 0
- joint left_wheel_joint: axis 1 0 0 -> -1 0 0; origin xyz=-0.0815 -0.0875 0.0378 -> xyz=-0.0815 -0.0875 0.0378 rpy=0 0 0
- joint right_wheel_joint: axis 1 0 0 -> -1 0 0; origin xyz=0.0815 -0.0875 0.0378 -> xyz=0.0815 -0.0875 0.0378 rpy=0 0 0

Commit message: Works

File: knight_description/urdf/knight.urdf (robot description, URDF)
Before this commit: robot knight, 6 links, 5 joints
Links:
- link base_link: mass 4 -> 7.7
- link left_wheel_link: mass 0.5 -> 1
- link right_wheel_link: mass 0.5 -> 1
